File: Panel/gategrinder_panel/gategrinder_panel.kicad_pcb (KiCad board)
At the start: 2 copper layers, 100 x 200 mm, 19 parts

Commit message: JLCJLCJLCJLC
Other:
- board text added: "JLCJLCJLCJLC"
Changed lines of the file:
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@@
   (general
     (thickness 1.6)
-    (drawings 4)
+    (drawings 5)
     (tracks 0)
     (zones 0)
@@
       (net 1 GND))
   )
+  (gr_text JLCJLCJLCJLC (at 141 192) (layer B.SilkS)
+    (effects (font (size 1 1) (thickness 0.16)) (justify mirror))
+  )
   (gr_line (start 90 200) (end 90 0) (layer Edge.Cuts) (width 0.05))

Commit message: Panel revision
Parts:
- moved H10 8.00 mm to (115.0, 95.3)
- moved H11 8.00 mm to (102.5, 160.5)
- moved H13 8.00 mm to (127.5, 175.5)
- moved H14 8.00 mm to (152.5, 95.5)
- moved H16 8.00 mm to (177.5, 175.5)
- moved H17 8.00 mm to (177.5, 95.5)
- moved H18 8.00 mm to (102.5, 175.5)
- moved H2 8.00 mm to (165.0, 132.9)
- moved H3 8.00 mm to (115.0, 133.0)
- moved H4 8.00 mm to (177.5, 45.4)
- moved H5 8.00 mm to (115.0, 45.5)
- moved H6 8.00 mm to (127.5, 160.5)
- moved H8 8.00 mm to (152.5, 175.5)
- moved H9 8.00 mm to (152.5, 45.4)
