File: PCB/v1/gategrinder_v1.kicad_pcb (KiCad board)
At the start: 2 copper layers, 196 x 96 mm, 72 parts, among them J1 EURO_PWR_2x5, J10 AudioJack3_SwitchTR, J3 Conn_01x14, J6 AudioJack3_SwitchTR, J7 AudioJack3_SwitchTR, J8 AudioJack3_SwitchTR, J9 AudioJack3_SwitchTR, Q1 BC547, Q2 BC547, Q3 BC547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

Commit message: NA556 -> NE556N
Parts:
- U1: value NA556 -> NE556N
Changed lines of the file:
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@@
     (46 B.CrtYd user)
     (47 F.CrtYd user)
-    (48 B.Fab user hide)
-    (49 F.Fab user hide)
+    (48 B.Fab user)
+    (49 F.Fab user)
   )
   (setup
@@
       (effects (font (size 1 1) (thickness 0.15)) (justify mirror))
     )
-    (fp_text value NA556 (at 3.81 -17.57 90) (layer B.Fab)
-      (effects (font (size 1 1) (thickness 0.15)) (justify mirror))
-    )
+    (fp_text value NE556N (at 3.81 -17.57 90) (layer B.Fab)
+      (effects (font (size 1 1) (thickness 0.15)) (justify mirror))
+    )
